File: koeg-board-pcb.kicad_pcb (KiCad board)
At the start: 2 copper layers, 10 parts, among them SW1 SW_Push_45deg, SW2 SW_Push_45deg, SW3 SW_Push_45deg, SW4 SW_Push_45deg, SW5 SW_Push_45deg, SW6 SW_Push_45deg, SW7 SW_Push_45deg, SW8 SW_Push_45deg, SW9 SW_Push_45deg, U1 STM32F730V8Tx

Commit message: before auto route
Parts:
- added AE1: PCB_Antenna, pcb_ant:pcb_antenna, B.Cu at (132.9, 122.5)
- added C1: 12pF, Capacitor_SMD:C_0402_1005Metric, B.Cu at (142.1, 119.5)
- added C10: 1pF, Capacitor_SMD:C_0402_1005Metric, B.Cu at (137.3, 121.3)
- added C11: 1.2pF, Capacitor_SMD:C_0402_1005Metric, B.Cu at (135.3, 121.1)
- added C12: 4.7uF, Capacitor_SMD:C_0402_1005Metric, B.Cu at (128.5, 108.7)
- added C13: 4.7uF, Capacitor_SMD:C_0402_1005Metric, B.Cu at (141.8, 107.1)
- added C14: 1uF, Capacitor_SMD:C_0402_1005Metric, B.Cu at (143.3, 96.6)
- added C15: 1uF, Capacitor_SMD:C_0402_1005Metric, B.Cu at (137.8, 96.5)
- added C16: 100nF, Capacitor_SMD:C_0402_1005Metric, B.Cu at (75.3, 116.2)
- added C2: 12pF, Capacitor_SMD:C_0402_1005Metric, B.Cu at (144.3, 116.9)
- added C3: 100nF, Capacitor_SMD:C_0402_1005Metric, B.Cu at (131.3, 105.1)
- added C4: 100pF, Capacitor_SMD:C_0402_1005Metric, B.Cu at (142.8, 107.8)
- added C5: 1uF, Capacitor_SMD:C_0402_1005Metric, B.Cu at (129.2, 119.1)
- added C6: 47nF, Capacitor_SMD:C_0402_1005Metric, B.Cu at (129.2, 118.2)
- added C7: 820pF, Capacitor_SMD:C_0402_1005Metric, B.Cu at (144.1, 115.2)
- added C8: 4.7uF, Capacitor_SMD:C_0402_1005Metric, B.Cu at (132.6, 109.7)
- added C9: 4.7uF, Capacitor_SMD:C_0402_1005Metric, B.Cu at (120.7, 117.3)
- added D1: 1N5819, Diode_SMD:D_SOD-123, B.Cu at (42.2, 70.1)
- added D10: 1N5819, Diode_SMD:D_SOD-123, B.Cu at (96.2, 81.4)
- added D11: 1N5819, Diode_SMD:D_SOD-123, B.Cu at (114.2, 87.1)
- added D12: 1N5819, Diode_SMD:D_SOD-123, B.Cu at (42.2, 104.1)
- added D13: 1N5819, Diode_SMD:D_SOD-123, B.Cu at (42.2, 121.1)
- added D14: 1N5819, Diode_SMD:D_SOD-123, B.Cu at (60.2, 98.4)
- added D15: 1N5819, Diode_SMD:D_SOD-123, B.Cu at (60.2, 115.4)
- added D16: 1N5819, Diode_SMD:D_SOD-123, B.Cu at (78.2, 92.8)
- added D17: 1N5819, Diode_SMD:D_SOD-123, B.Cu at (78.2, 109.8)
- added D18: 1N5819, Diode_SMD:D_SOD-123, B.Cu at (96.2, 98.4)
- added D19: 1N5819, Diode_SMD:D_SOD-123, B.Cu at (96.2, 115.4)
- added D2: 1N5819, Diode_SMD:D_SOD-123, B.Cu at (129.5, 97.4)
- added D20: 1N5819, Diode_SMD:D_SOD-123, B.Cu at (114.2, 104.1)
- added D21: 1N5819, Diode_SMD:D_SOD-123, B.Cu at (114.2, 121.1)
- added D22: 1N5819, Diode_SMD:D_SOD-123, B.Cu at (128.5, 102.1)
- added D23: WS2812B-2020, LED_SMD:LED_WS2812B_PLCC4_5.0x5.0mm_P3.2mm, B.Cu at (122.3, 121.5)
- added D24: WS2812B-2020, LED_SMD:LED_WS2812B_PLCC4_5.0x5.0mm_P3.2mm, B.Cu at (104.2, 115.9)
- added D25: WS2812B-2020, LED_SMD:LED_WS2812B_PLCC4_5.0x5.0mm_P3.2mm, B.Cu at (86.2, 110.2)
- added D26: WS2812B-2020, LED_SMD:LED_WS2812B_PLCC4_5.0x5.0mm_P3.2mm, B.Cu at (68.2, 115.9)
- added D27: WS2812B-2020, LED_SMD:LED_WS2812B_PLCC4_5.0x5.0mm_P3.2mm, B.Cu at (50.2, 121.5)
- added D28: WS2812B-2020, LED_SMD:LED_WS2812B_PLCC4_5.0x5.0mm_P3.2mm, B.Cu at (122.3, 104.5)
- added D29: WS2812B-2020, LED_SMD:LED_WS2812B_PLCC4_5.0x5.0mm_P3.2mm, B.Cu at (104.3, 98.8)
- added D3: 1N5819, Diode_SMD:D_SOD-123, B.Cu at (60.2, 64.4)
- added D30: WS2812B-2020, LED_SMD:LED_WS2812B_PLCC4_5.0x5.0mm_P3.2mm, B.Cu at (86.2, 93.2)
- added D31: WS2812B-2020, LED_SMD:LED_WS2812B_PLCC4_5.0x5.0mm_P3.2mm, B.Cu at (68.2, 98.8)
- added D32: WS2812B-2020, LED_SMD:LED_WS2812B_PLCC4_5.0x5.0mm_P3.2mm, B.Cu at (50.2, 104.5)
- added D33: WS2812B-2020, LED_SMD:LED_WS2812B_PLCC4_5.0x5.0mm_P3.2mm, B.Cu at (122.2, 87.5)
- added D34: WS2812B-2020, LED_SMD:LED_WS2812B_PLCC4_5.0x5.0mm_P3.2mm, B.Cu at (104.3, 81.8)
- added D35: WS2812B-2020, LED_SMD:LED_WS2812B_PLCC4_5.0x5.0mm_P3.2mm, B.Cu at (86.3, 76.2)
- added D36: WS2812B-2020, LED_SMD:LED_WS2812B_PLCC4_5.0x5.0mm_P3.2mm, B.Cu at (68.3, 81.8)
- added D37: WS2812B-2020, LED_SMD:LED_WS2812B_PLCC4_5.0x5.0mm_P3.2mm, B.Cu at (50.2, 87.5)
- added D38: WS2812B-2020, LED_SMD:LED_WS2812B_PLCC4_5.0x5.0mm_P3.2mm, B.Cu at (122.2, 70.5)
- added D39: WS2812B-2020, LED_SMD:LED_WS2812B_PLCC4_5.0x5.0mm_P3.2mm, B.Cu at (104.2, 64.8)
- added D4: 1N5819, Diode_SMD:D_SOD-123, B.Cu at (78.2, 58.8)
- added D40: WS2812B-2020, LED_SMD:LED_WS2812B_PLCC4_5.0x5.0mm_P3.2mm, B.Cu at (86.2, 59.2)
- added D41: WS2812B-2020, LED_SMD:LED_WS2812B_PLCC4_5.0x5.0mm_P3.2mm, B.Cu at (68.2, 64.8)
- added D42: WS2812B-2020, LED_SMD:LED_WS2812B_PLCC4_5.0x5.0mm_P3.2mm, B.Cu at (50.3, 70.5)
- added D5: 1N5819, Diode_SMD:D_SOD-123, B.Cu at (96.2, 64.4)
- added D6: 1N5819, Diode_SMD:D_SOD-123, B.Cu at (114.2, 70.1)
- added D7: 1N5819, Diode_SMD:D_SOD-123, B.Cu at (42.2, 87.1)
- added D8: 1N5819, Diode_SMD:D_SOD-123, B.Cu at (60.2, 81.4)
- added D9: 1N5819, Diode_SMD:D_SOD-123, B.Cu at (78.2, 75.8)
- added F1: 500mA, Fuse:Fuse_0603_1608Metric, B.Cu at (129.2, 110.1)
- added H1: MountingHole, MountingHole:MountingHole_2mm, B.Cu at (56.1, 68.2)
- added H2: MountingHole, MountingHole:MountingHole_2mm, B.Cu at (74.3, 84.8)
- added H3: MountingHole, MountingHole:MountingHole_2mm, B.Cu at (109.2, 103.3)
- added H4: MountingHole, MountingHole:MountingHole_2mm, B.Cu at (54.7, 108.8)
- added H5: MountingHole, MountingHole:MountingHole_2mm, B.Cu at (109.3, 69.2)
- added J1: Conn_01x02, Connector_PinHeader_1.00mm:PinHeader_1x02_P1.00mm_Vertical, F.Cu at (106.8, 120.7)
- added J2: USB_C_Receptacle_USB2.0_14P, Connector_USB:USB_C_Receptacle_G-Switch_GT-USB-7010ASV, B.Cu at (113.9, 51.8)
- added J3: SWD_Connector, Connector_PinHeader_1.00mm:PinHeader_1x04_P1.00mm_Vertical, F.Cu at (86.8, 115.2)
- added L1: 10uH, Inductor_SMD:L_0201_0603Metric, B.Cu at (129.4, 116.5)
- added L2: 15nH, Inductor_SMD:L_0201_0603Metric, B.Cu at (129.4, 117.3)
- added L3: 10uH, Inductor_SMD:L_0201_0603Metric, B.Cu at (130.9, 107.0)
- added L4: 4.7nH, Inductor_SMD:L_0201_0603Metric, B.Cu at (136.8, 122.1)
- added L5: 2.2nH, Inductor_SMD:L_0201_0603Metric, B.Cu at (135.3, 122.1)
- added Q1: BSS138, Package_TO_SOT_SMD:SOT-23, B.Cu at (111.4, 113.7)
- added R1: 5.1k, Resistor_SMD:R_0201_0603Metric, B.Cu at (90.6, 53.6)
- added R2: 5.1k, Resistor_SMD:R_0201_0603Metric, B.Cu at (90.7, 55.8)
- added R3: 2M, Resistor_SMD:R_0201_0603Metric, B.Cu at (140.9, 98.5)
- added R4: 810K, Resistor_SMD:R_0201_0603Metric, B.Cu at (141.0, 97.8)
- added R5: 10K, Resistor_SMD:R_0201_0603Metric, B.Cu at (114.0, 113.8)
- added R6: 10K, Resistor_SMD:R_0201_0603Metric, B.Cu at (113.5, 115.9)
- added R7: 100K, Resistor_SMD:R_0201_0603Metric, B.Cu at (136.8, 109.4)
- added SW10: SW_Push, PCM_Switch_Keyboard_Hotswap_Kailh:SW_Hotswap_Kailh_Choc_V1V2_1.00u, F.Cu at (81.1, 71.3)
- added SW11: SW_Push, PCM_Switch_Keyboard_Hotswap_Kailh:SW_Hotswap_Kailh_Choc_V1V2_1.00u, F.Cu at (99.1, 77.0)
- added SW12: SW_Push, PCM_Switch_Keyboard_Hotswap_Kailh:SW_Hotswap_Kailh_Choc_V1V2_1.00u, F.Cu at (117.1, 82.7)
- added SW13: SW_Push, PCM_Switch_Keyboard_Hotswap_Kailh:SW_Hotswap_Kailh_Choc_V1V2_1.00u, F.Cu at (45.1, 99.7)
- added SW14: SW_Push, PCM_Switch_Keyboard_Hotswap_Kailh:SW_Hotswap_Kailh_Choc_V1V2_1.00u, F.Cu at (45.1, 116.7)
- added SW15: SW_Push, PCM_Switch_Keyboard_Hotswap_Kailh:SW_Hotswap_Kailh_Choc_V1V2_1.00u, F.Cu at (63.1, 94.0)
- added SW16: SW_Push, PCM_Switch_Keyboard_Hotswap_Kailh:SW_Hotswap_Kailh_Choc_V1V2_1.00u, F.Cu at (63.1, 111.0)
- added SW17: SW_Push, PCM_Switch_Keyboard_Hotswap_Kailh:SW_Hotswap_Kailh_Choc_V1V2_1.00u, F.Cu at (81.1, 88.3)
- added SW18: SW_Push, PCM_Switch_Keyboard_Hotswap_Kailh:SW_Hotswap_Kailh_Choc_V1V2_1.00u, F.Cu at (81.1, 105.3)
- added SW19: SW_Push, PCM_Switch_Keyboard_Hotswap_Kailh:SW_Hotswap_Kailh_Choc_V1V2_1.00u, F.Cu at (99.1, 94.0)
- added SW20: SW_Push, PCM_Switch_Keyboard_Hotswap_Kailh:SW_Hotswap_Kailh_Choc_V1V2_1.00u, F.Cu at (99.1, 111.0)
- added SW21: SW_Push, PCM_Switch_Keyboard_Hotswap_Kailh:SW_Hotswap_Kailh_Choc_V1V2_1.00u, F.Cu at (117.1, 99.7)
- added SW22: SW_Push, PCM_Switch_Keyboard_Hotswap_Kailh:SW_Hotswap_Kailh_Choc_V1V2_1.00u, F.Cu at (117.1, 116.7)
- added SW23: SW_Push, PCM_Switch_Keyboard_Hotswap_Kailh:SW_Hotswap_Kailh_Choc_V1V2_1.75u_90deg, F.Cu at (134.6, 106.9)
- added U2: AMS1117-5.0, Package_TO_SOT_SMD:SOT-223-3_TabPin2, B.Cu at (140.7, 92.4)
- added U3: USBLC6-2SC6, Package_TO_SOT_SMD:SOT-23-6, B.Cu at (111.8, 96.3)
- added Y1: Crystal_GND2, Crystal:Crystal_SMD_2016-4Pin_2.0x1.6mm, B.Cu at (144.4, 118.9)
- SW1, SW4, SW5, SW6, SW7, SW8, SW9: value SW_Push_45deg -> SW_Push; footprint PCM_Switch_Keyboard_Hotswap_Kailh:SW_Hotswap_Kailh_Choc_V2_Plated -> PCM_Switch_Keyboard_Hotswap_Kailh:SW_Hotswap_Kailh_Choc_V1V2_1.00u
- SW2: value SW_Push_45deg -> Reset Button; footprint PCM_Switch_Keyboard_Hotswap_Kailh:SW_Hotswap_Kailh_Choc_V2_Plated -> Button_Switch_SMD:SW_SPST_TL3342; moved to B.Cu
- SW3: value SW_Push_45deg -> SW_On_Off; footprint PCM_Switch_Keyboard_Hotswap_Kailh:SW_Hotswap_Kailh_Choc_V2_Plated -> Button_Switch_THT:SW_CK_JS202011AQN_DPDT_Angled; moved to B.Cu
- U1: value STM32F730V8Tx -> nRF52840; footprint Package_QFP:LQFP-100_14x14mm_P0.5mm -> Package_DFN_QFN:Nordic_AQFN-73-1EP_7x7mm_P0.5mm; moved to B.Cu
- moved SW8 167.4 mm to (45.1, 82.7)
- moved SW9 151.1 mm to (63.1, 77.0)
- moved SW4 132.7 mm to (63.1, 60.0)
- moved SW2 131.9 mm to (80.1, 116.2), turned to 180 degrees
- moved SW1 128.9 mm to (45.1, 65.7)
- moved SW5 121.5 mm to (81.1, 54.3)
- moved SW6 110.4 mm to (99.1, 60.0)
- moved U1 105.6 mm to (138.7, 114.4)
- moved SW7 95.4 mm to (117.1, 65.7)
- moved SW3 71.0 mm to (128.5, 92.4)
Connections:
- SW1 pad 1: unconnected-(SW1-Pad1) -> Net-(D1-A)
- SW1 pad 2: GND -> /COL0
- SW2 pad 1: unconnected-(SW2-Pad1) -> /RESET
- SW3 pad 2: GND -> VBAT
- SW4 pad 1: unconnected-(SW4-Pad1) -> Net-(D3-A)
- SW4 pad 2: GND -> /COL1
- SW5 pad 1: unconnected-(SW5-Pad1) -> Net-(D4-A)
- SW5 pad 2: GND -> /COL2
- SW6 pad 1: unconnected-(SW6-Pad1) -> Net-(D5-A)
- SW6 pad 2: GND -> /COL3
- SW7 pad 1: unconnected-(SW7-Pad1) -> Net-(D6-A)
- SW7 pad 2: GND -> /COL4
- SW8 pad 1: unconnected-(SW8-Pad1) -> Net-(D7-A)
- SW8 pad 2: GND -> /COL0
- SW9 pad 1: unconnected-(SW9-Pad1) -> Net-(D8-A)
- SW9 pad 2: GND -> /COL1
Routing:
- net /D-: track 0.00 -> 70.6 mm, vias 0 -> 2
- net /D+: track 0.00 -> 70.6 mm, vias 0 -> 2
- net GND: track 0.00 -> 6.74 mm, vias 0 -> 2
- net /DEC3: track 0.00 -> 0.11 mm, vias 0 -> 1
- net /DEC4: track 0.00 -> 0.05 mm, vias 0 -> 2
- net V_SYS: track 0.00 -> 0.04 mm, vias 0 -> 5
- net /XC1: track 0.00 -> 0.03 mm, vias 0 -> 1
- net /RESET: track 0.00 -> 0.03 mm, vias 0 -> 1
- net 3.2V-5V: track 0.00 -> 0.03 mm, vias 0 -> 1
- net /ANT: track 0.00 -> 0.03 mm, vias 0 -> 1
- net /DECUSB: track 0.00 -> 0.03 mm, vias 0 -> 1
- net /DCC: track 0.00 -> 0.02 mm, vias 0 -> 1
- net /DCCH: track 0.00 -> 0.02 mm, vias 0 -> 1
- net /ROW0: track 0.00 -> 0.02 mm, vias 0 -> 1
- net LED_PIN: track 0.00 -> 0.01 mm, vias 0 -> 1
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Other:
- board outline added: 112.2 x 84 mm

Commit message: autorouted
Routing:
- net GND: track 6.74 -> 581.3 mm, vias 2 -> 14
- net LED_5V: track 0.00 -> 420.4 mm, vias 0 -> 4
- net /ROW0: track 0.02 -> 191.6 mm, vias 1 -> 6
- net /COL2: track 0.00 -> 168.6 mm, vias 0 -> 4
- net /ROW1: track 0.01 -> 167.1 mm, vias 1 -> 7
- net /COL0: track 0.00 -> 162.4 mm, vias 1 -> 5
- net /COL1: track 0.00 -> 161.2 mm, vias 1 -> 8
- net /COL3: track 0.01 -> 123.6 mm, vias 1 -> 4
- net /ROW2: track 0.00 -> 122.1 mm, vias 1 -> 5
- net V_SYS: track 0.04 -> 118.1 mm, vias 5 -> 13
- net /RESET: track 0.03 -> 96.3 mm, vias 1 -> 6
- net VBUS: track 0.00 -> 93.1 mm, vias 0 -> 6
- net /ROW3: track 0.01 -> 89.6 mm, vias 1 -> 4
- net /COL4: track 0.00 -> 88.5 mm, vias 1 -> 4
- net /SWDIO: track 0.00 -> 84.7 mm, vias 1 -> 6
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
Commit message: one side done
Parts:
- removed Y1: Crystal_GND2, Crystal:Crystal_SMD_2016-4Pin_2.0x1.6mm
- added Y2: JYJE 2TJ432000NYFBC, Crystal:Crystal_SMD_2520-4Pin_2.5x2.0mm, B.Cu at (143.5, 120.8)
- J2: footprint Connector_USB:USB_C_Receptacle_G-Switch_GT-USB-7010ASV -> USB_Type_C:HRO-TYPE-C-31-M-12
- L1, L3: footprint Inductor_SMD:L_0201_0603Metric -> Inductor_SMD:L_1008_2520Metric
- R3: value 2M -> 10K
- R4: value 810K -> 10K
- moved L3 18.0 mm to (128.4, 124.8), turned to -90 degrees
- moved C3 9.64 mm to (129.8, 114.6), turned to 180 degrees
- moved C2 5.35 mm to (141.3, 121.3), turned to -90 degrees
- moved J2 3.82 mm to (113.9, 48.0)
- moved C1 3.06 mm to (144.6, 117.7)
- moved R4 2.73 mm to (143.2, 99.3), turned to 180 degrees
- moved L1 2.70 mm to (126.8, 115.6)
- moved U3 2.09 mm to (110.0, 95.2), turned to 180 degrees
- moved C8 1.68 mm to (132.7, 111.4), turned to 90 degrees
- moved R7 1.60 mm to (137.9, 108.3)
- moved R3 1.21 mm to (139.7, 98.5)
- moved C10 0.17 mm to (137.3, 121.1)
- moved L4 0.06 mm to (136.8, 122.1)
- moved L5 0.06 mm to (135.3, 122.1)
Connections:
- U1 pad AD12: unconnected-(U1-P0.17-PadAD12) -> /RESET
- U1 pad AD8: unconnected-(U1-P0.13-PadAD8) -> /DECUSB
Routing:
- net GND: track 581.3 -> 654.4 mm, vias 14 -> 22
- net /ROW3: track 89.6 -> 126.5 mm, vias 4 -> 5
- net V_SYS: track 118.1 -> 142.3 mm, vias 13 -> 12
- net /DCCH: track 7.90 -> 22.6 mm, vias 2 -> 4
- net LED_5V: track 420.4 -> 433.9 mm, vias 4 -> 6
- net /DECUSB: track 0.03 -> 8.81 mm, vias 1 -> 2
- net /DEC1: track 0.01 -> 6.88 mm, vias 1 -> 2
- net VBAT: track 83.2 -> 88.5 mm
- net /D+: track 80.1 -> 85.2 mm, vias 3 -> 5
- net /BT_PIN: track 25.8 -> 30.4 mm
- net Net-(L1-Pad2): track 0.81 -> 4.99 mm
- net /XC1: track 3.97 -> 8.07 mm, vias 1 -> 0
- net 5V: track 62.0 -> 66.1 mm
- net /SWDCLK: track 67.3 -> 71.2 mm
- net /DEC4: track 30.4 -> 33.5 mm
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Other:
- board size 112.2 x 84 mm -> 112.5 x 84.2 mm

Commit message: reassigned basic components, now comes the leds
Parts:
- added AE2: PCB_Antenna, pcb_ant:pcb_antenna, F.Cu at (422.7, 91.1)
- added C17: 4.7uF, Capacitor_SMD:C_0402_1005Metric, F.Cu at (421.0, 125.2)
- added C18: 4.7uF, Capacitor_SMD:C_0402_1005Metric, F.Cu at (421.0, 127.1)
- added C19: 100nF, Capacitor_SMD:C_0402_1005Metric, F.Cu at (421.0, 129.1)
- added C20: 100pF, Capacitor_SMD:C_0402_1005Metric, F.Cu at (421.0, 131.1)
- added C21: 820pF, Capacitor_SMD:C_0402_1005Metric, F.Cu at (421.0, 133.1)
- added C22: 100nF, Capacitor_SMD:C_0402_1005Metric, F.Cu at (423.9, 125.2)
- added C23: 1uF, Capacitor_SMD:C_0402_1005Metric, F.Cu at (423.9, 127.1)
- added C24: 47nF, Capacitor_SMD:C_0402_1005Metric, F.Cu at (423.9, 129.1)
- added C25: 4.7uF, Capacitor_SMD:C_0402_1005Metric, F.Cu at (423.9, 131.1)
- added C26: 4.7uF, Capacitor_SMD:C_0402_1005Metric, F.Cu at (423.9, 133.1)
- added C27: 12pF, Capacitor_SMD:C_0402_1005Metric, F.Cu at (426.8, 125.2)
- added C28: 12pF, Capacitor_SMD:C_0402_1005Metric, F.Cu at (426.8, 127.1)
- added C29: 1pF, Capacitor_SMD:C_0402_1005Metric, F.Cu at (426.8, 129.1)
- added C30: 1.2pF, Capacitor_SMD:C_0402_1005Metric, F.Cu at (426.8, 131.1)
- added C31: 1uF, Capacitor_SMD:C_0402_1005Metric, F.Cu at (394.8, 160.4)
- added C32: 1uF, Capacitor_SMD:C_0402_1005Metric, F.Cu at (394.8, 162.4)
- added D23: SK6812MINI, Keebio_Parts:SK6812-MINI-E, B.Cu at (120.8, 129.3)
- added D24: SK6812MINI, Keebio_Parts:SK6812-MINI-E, F.Cu at (349.3, 143.6)
- added D25: SK6812MINI, Keebio_Parts:SK6812-MINI-E, F.Cu at (349.3, 148.2)
- added D26: SK6812MINI, Keebio_Parts:SK6812-MINI-E, F.Cu at (349.3, 152.8)
- added D27: SK6812MINI, Keebio_Parts:SK6812-MINI-E, B.Cu at (349.8, 157.4)
- added D28: SK6812MINI, Keebio_Parts:SK6812-MINI-E, F.Cu at (357.1, 138.9)
- added D29: SK6812MINI, Keebio_Parts:SK6812-MINI-E, F.Cu at (357.1, 143.6)
- added D30: SK6812MINI, Keebio_Parts:SK6812-MINI-E, F.Cu at (357.1, 148.2)
- added D31: SK6812MINI, Keebio_Parts:SK6812-MINI-E, F.Cu at (357.1, 152.8)
- added D32: SK6812MINI, Keebio_Parts:SK6812-MINI-E, F.Cu at (357.1, 157.4)
- added D33: SK6812MINI, Keebio_Parts:SK6812-MINI-E, F.Cu at (364.9, 138.9)
- added D34: SK6812MINI, Keebio_Parts:SK6812-MINI-E, F.Cu at (364.9, 143.6)
- added D35: SK6812MINI, Keebio_Parts:SK6812-MINI-E, F.Cu at (364.9, 148.2)
- added D36: SK6812MINI, Keebio_Parts:SK6812-MINI-E, F.Cu at (364.9, 152.8)
- added D37: SK6812MINI, Keebio_Parts:SK6812-MINI-E, F.Cu at (364.9, 157.4)
- added D38: SK6812MINI, Keebio_Parts:SK6812-MINI-E, F.Cu at (372.7, 138.9)
- added D39: SK6812MINI, Keebio_Parts:SK6812-MINI-E, F.Cu at (372.7, 143.6)
- added D40: SK6812MINI, Keebio_Parts:SK6812-MINI-E, F.Cu at (372.7, 148.2)
- added D41: SK6812MINI, Keebio_Parts:SK6812-MINI-E, F.Cu at (372.7, 152.8)
- added D42: SK6812MINI, Keebio_Parts:SK6812-MINI-E, F.Cu at (372.7, 157.4)
- added D43: 1N5819, Diode_SMD:D_SOD-123, F.Cu at (422.5, 60.3)
- added D44: 1N5819, Diode_SMD:D_SOD-123, F.Cu at (422.5, 63.7)
- added D45: 1N5819, Diode_SMD:D_SOD-123, F.Cu at (422.5, 67.0)
- added D46: 1N5819, Diode_SMD:D_SOD-123, F.Cu at (422.5, 70.4)
- added D47: 1N5819, Diode_SMD:D_SOD-123, F.Cu at (422.5, 73.7)
- added D48: 1N5819, Diode_SMD:D_SOD-123, F.Cu at (422.5, 77.1)
- added D49: 1N5819, Diode_SMD:D_SOD-123, F.Cu at (422.5, 80.4)
- added D50: 1N5819, Diode_SMD:D_SOD-123, F.Cu at (422.5, 83.8)
- added D51: 1N5819, Diode_SMD:D_SOD-123, F.Cu at (428.3, 60.3)
- added D52: 1N5819, Diode_SMD:D_SOD-123, F.Cu at (428.3, 63.7)
- added D53: 1N5819, Diode_SMD:D_SOD-123, F.Cu at (428.3, 67.0)
- added D54: 1N5819, Diode_SMD:D_SOD-123, F.Cu at (428.3, 70.4)
- added D55: 1N5819, Diode_SMD:D_SOD-123, F.Cu at (428.3, 73.7)
- added D56: 1N5819, Diode_SMD:D_SOD-123, F.Cu at (428.3, 77.1)
- added D57: 1N5819, Diode_SMD:D_SOD-123, F.Cu at (428.3, 80.4)
- added D58: 1N5819, Diode_SMD:D_SOD-123, F.Cu at (428.3, 83.8)
- added D59: 1N5819, Diode_SMD:D_SOD-123, F.Cu at (434.1, 60.3)
- added D60: 1N5819, Diode_SMD:D_SOD-123, F.Cu at (434.1, 63.7)
- added D61: 1N5819, Diode_SMD:D_SOD-123, F.Cu at (434.1, 67.0)
- added D62: 1N5819, Diode_SMD:D_SOD-123, F.Cu at (434.1, 70.4)
- added D63: 1N5819, Diode_SMD:D_SOD-123, F.Cu at (434.1, 73.7)
- added D64: 1N5819, Diode_SMD:D_SOD-123, F.Cu at (434.1, 77.1)
- added D65: SK6812MINI, Keebio_Parts:SK6812-MINI-E, F.Cu at (382.5, 138.9)
- added D66: SK6812MINI, Keebio_Parts:SK6812-MINI-E, F.Cu at (382.5, 143.6)
- added D67: SK6812MINI, Keebio_Parts:SK6812-MINI-E, F.Cu at (382.5, 148.2)
- added D68: SK6812MINI, Keebio_Parts:SK6812-MINI-E, F.Cu at (382.5, 152.8)
- added D69: SK6812MINI, Keebio_Parts:SK6812-MINI-E, F.Cu at (382.5, 157.4)
- added D70: SK6812MINI, Keebio_Parts:SK6812-MINI-E, F.Cu at (390.3, 138.9)
- added D71: SK6812MINI, Keebio_Parts:SK6812-MINI-E, F.Cu at (390.3, 143.6)
- added D72: SK6812MINI, Keebio_Parts:SK6812-MINI-E, F.Cu at (390.3, 148.2)
- added D73: SK6812MINI, Keebio_Parts:SK6812-MINI-E, F.Cu at (390.3, 152.8)
- added D74: SK6812MINI, Keebio_Parts:SK6812-MINI-E, F.Cu at (390.3, 157.4)
- added D75: SK6812MINI, Keebio_Parts:SK6812-MINI-E, F.Cu at (398.1, 138.9)
- added D76: SK6812MINI, Keebio_Parts:SK6812-MINI-E, F.Cu at (398.1, 143.6)
- added D77: SK6812MINI, Keebio_Parts:SK6812-MINI-E, F.Cu at (398.1, 148.2)
- added D78: SK6812MINI, Keebio_Parts:SK6812-MINI-E, F.Cu at (398.1, 152.8)
- added D79: SK6812MINI, Keebio_Parts:SK6812-MINI-E, F.Cu at (398.1, 157.4)
- added D80: SK6812MINI, Keebio_Parts:SK6812-MINI-E, F.Cu at (405.9, 138.9)
- added D81: SK6812MINI, Keebio_Parts:SK6812-MINI-E, F.Cu at (405.9, 143.6)
- added D82: SK6812MINI, Keebio_Parts:SK6812-MINI-E, F.Cu at (405.9, 148.2)
- added D83: SK6812MINI, Keebio_Parts:SK6812-MINI-E, F.Cu at (405.9, 152.8)
- added D84: SK6812MINI, Keebio_Parts:SK6812-MINI-E, F.Cu at (405.9, 157.4)
- added F2: 500mA, Fuse:Fuse_0603_1608Metric, F.Cu at (430.5, 51.3)
- added H10: MountingHole, MountingHole:MountingHole_2mm, F.Cu at (422.4, 55.9)
- added H6: MountingHole, MountingHole:MountingHole_2mm, F.Cu at (422.4, 33.7)
- added H7: MountingHole, MountingHole:MountingHole_2mm, F.Cu at (422.4, 39.2)
- added H8: MountingHole, MountingHole:MountingHole_2mm, F.Cu at (422.4, 44.8)
- added H9: MountingHole, MountingHole:MountingHole_2mm, F.Cu at (422.4, 50.3)
- added J4: Conn_01x02, Connector_PinHeader_1.00mm:PinHeader_1x02_P1.00mm_Vertical, F.Cu at (426.8, 51.6)
- added J5: SWD_Connector, Connector_PinHeader_1.00mm:PinHeader_1x04_P1.00mm_Vertical, F.Cu at (431.8, 39.5)
- added J6: USB_C_Receptacle_USB2.0_14P, USB_Type_C:HRO-TYPE-C-31-M-12, F.Cu at (427.3, 101.1)
- added L10: 2.2nH, Inductor_SMD:L_0201_0603Metric, F.Cu at (420.8, 96.5)
- added L6: 10uH, Inductor_SMD:L_1008_2520Metric, F.Cu at (427.6, 39.8)
- added L7: 15nH, Inductor_SMD:L_0201_0603Metric, F.Cu at (420.8, 93.0)
- added L8: 10uH, Inductor_SMD:L_1008_2520Metric, F.Cu at (427.6, 43.6)
- added L9: 4.7nH, Inductor_SMD:L_0201_0603Metric, F.Cu at (420.8, 94.8)
- added Q2: BSS138, Package_TO_SOT_SMD:SOT-23, F.Cu at (390.9, 161.8)
- added R10: 10K, Resistor_SMD:R_0201_0603Metric, F.Cu at (420.8, 101.8)
- added R11: 5.1k, Resistor_SMD:R_0201_0603Metric, F.Cu at (420.8, 103.5)
- added R12: 5.1k, Resistor_SMD:R_0201_0603Metric, F.Cu at (420.8, 105.3)
- added R13: 10K, Resistor_SMD:R_0201_0603Metric, F.Cu at (394.5, 164.3)
- added R14: 10K, Resistor_SMD:R_0201_0603Metric, F.Cu at (394.5, 166.0)
- added R8: 100K, Resistor_SMD:R_0201_0603Metric, F.Cu at (420.8, 98.3)
- added R9: 10K, Resistor_SMD:R_0201_0603Metric, F.Cu at (420.8, 100.0)
- added SW24: SW_On_Off, Button_Switch_THT:SW_CK_JS202011AQN_DPDT_Angled, F.Cu at (422.4, 107.6)
- added SW25: SW_Push, PCM_Switch_Keyboard_Hotswap_Kailh:SW_Hotswap_Kailh_Choc_V1V2_1.00u, F.Cu at (353.6, 39.9)
- added SW26: SW_Push, PCM_Switch_Keyboard_Hotswap_Kailh:SW_Hotswap_Kailh_Choc_V1V2_1.00u, F.Cu at (353.6, 57.1)
- added SW27: SW_Push, PCM_Switch_Keyboard_Hotswap_Kailh:SW_Hotswap_Kailh_Choc_V1V2_1.00u, F.Cu at (353.6, 74.4)
- added SW28: SW_Push, PCM_Switch_Keyboard_Hotswap_Kailh:SW_Hotswap_Kailh_Choc_V1V2_1.00u, F.Cu at (353.6, 91.6)
- added SW29: SW_Push, PCM_Switch_Keyboard_Hotswap_Kailh:SW_Hotswap_Kailh_Choc_V1V2_1.00u, F.Cu at (353.6, 108.9)
- added SW30: Reset Button, Button_Switch_SMD:SW_SPST_TL3342, F.Cu at (429.9, 34.4)
- added SW31: SW_Push, PCM_Switch_Keyboard_Hotswap_Kailh:SW_Hotswap_Kailh_Choc_V1V2_1.00u, F.Cu at (353.6, 126.1)
- added SW32: SW_Push, PCM_Switch_Keyboard_Hotswap_Kailh:SW_Hotswap_Kailh_Choc_V1V2_1.00u, F.Cu at (372.2, 39.9)
- added SW33: SW_Push, PCM_Switch_Keyboard_Hotswap_Kailh:SW_Hotswap_Kailh_Choc_V1V2_1.00u, F.Cu at (372.2, 57.1)
- added SW34: SW_Push, PCM_Switch_Keyboard_Hotswap_Kailh:SW_Hotswap_Kailh_Choc_V1V2_1.00u, F.Cu at (372.2, 74.4)
- added SW35: SW_Push, PCM_Switch_Keyboard_Hotswap_Kailh:SW_Hotswap_Kailh_Choc_V1V2_1.00u, F.Cu at (372.2, 91.6)
- added SW36: SW_Push, PCM_Switch_Keyboard_Hotswap_Kailh:SW_Hotswap_Kailh_Choc_V1V2_1.00u, F.Cu at (372.2, 108.9)
- added SW37: SW_Push, PCM_Switch_Keyboard_Hotswap_Kailh:SW_Hotswap_Kailh_Choc_V1V2_1.00u, F.Cu at (372.2, 126.1)
- added SW38: SW_Push, PCM_Switch_Keyboard_Hotswap_Kailh:SW_Hotswap_Kailh_Choc_V1V2_1.00u, F.Cu at (390.8, 39.9)
- added SW39: SW_Push, PCM_Switch_Keyboard_Hotswap_Kailh:SW_Hotswap_Kailh_Choc_V1V2_1.00u, F.Cu at (390.8, 57.1)
- added SW40: SW_Push, PCM_Switch_Keyboard_Hotswap_Kailh:SW_Hotswap_Kailh_Choc_V1V2_1.00u, F.Cu at (390.8, 74.4)
- added SW41: SW_Push, PCM_Switch_Keyboard_Hotswap_Kailh:SW_Hotswap_Kailh_Choc_V1V2_1.00u, F.Cu at (390.8, 91.6)
- added SW42: SW_Push, PCM_Switch_Keyboard_Hotswap_Kailh:SW_Hotswap_Kailh_Choc_V1V2_1.00u, F.Cu at (390.8, 108.9)
- added SW43: SW_Push, PCM_Switch_Keyboard_Hotswap_Kailh:SW_Hotswap_Kailh_Choc_V1V2_1.00u, F.Cu at (390.8, 126.1)
- added SW44: SW_Push, PCM_Switch_Keyboard_Hotswap_Kailh:SW_Hotswap_Kailh_Choc_V1V2_1.00u, F.Cu at (409.3, 39.9)
- added SW45: SW_Push, PCM_Switch_Keyboard_Hotswap_Kailh:SW_Hotswap_Kailh_Choc_V1V2_1.00u, F.Cu at (409.3, 57.1)
- added SW46: SW_Push, PCM_Switch_Keyboard_Hotswap_Kailh:SW_Hotswap_Kailh_Choc_V1V2_1.75u_90deg, F.Cu at (409.3, 74.4)
- added U4: nRF52840, Package_DFN_QFN:Nordic_AQFN-73-1EP_7x7mm_P0.5mm, F.Cu at (424.6, 119.2)
- added U5: USBLC6-2SC6, Package_TO_SOT_SMD:SOT-23-6, F.Cu at (427.7, 47.8)
- added U6: AMS1117-5.0, Package_TO_SOT_SMD:SOT-223-3_TabPin2, F.Cu at (383.5, 163.6)
- added Y2: JYJE 2TJ432000NYFBC, Crystal:Crystal_SMD_2520-4Pin_2.5x2.0mm, F.Cu at (432.5, 47.5)
- renumbered C12 to C1, C9 to C10, C1 to C11, C2 to C12, C10 to C13, C11 to C14, C14 to C15, C15 to C16, C16 to C2, C13 to C3, C3 to C4, C4 to C5, C7 to C6, C5 to C7, C6 to C8, C8 to C9, D14 to D13, D16 to D14, D18 to D15, D20 to D16, D13 to D17, D15 to D18, D17 to D19, D1 to D2, D19 to D20, J3 to J2, J2 to J3, R7 to R1, R4 to R2, R1 to R4, R2 to R5, R5 to R6, R6 to R7, SW3 to SW1, SW2 to SW1, SW15 to SW14, SW17 to SW15, SW19 to SW16, SW21 to SW17, SW14 to SW18, SW16 to SW19, SW18 to SW20, SW20 to SW21, SW1 to SW3, U3 to U2, U2 to U3, Y2 to Y1
Routing:
- net 3.2V-5V: track 26.5 -> 42.2 mm, vias 1 -> 3
- net Net-(D21-A): track 29.8 -> 17.6 mm
- net /DCCH: track 22.6 -> 23.2 mm

Commit message: placed leds
Parts:
- removed AE2: PCB_Antenna, pcb_ant:pcb_antenna
- removed C17, C18, C25, C26: 4.7uF, Capacitor_SMD:C_0402_1005Metric
- removed C19, C22: 100nF, Capacitor_SMD:C_0402_1005Metric
- removed C20: 100pF, Capacitor_SMD:C_0402_1005Metric
- removed C21: 820pF, Capacitor_SMD:C_0402_1005Metric
- removed C23, C31, C32: 1uF, Capacitor_SMD:C_0402_1005Metric
- removed C24: 47nF, Capacitor_SMD:C_0402_1005Metric
- removed C27, C28: 12pF, Capacitor_SMD:C_0402_1005Metric
- removed C29: 1pF, Capacitor_SMD:C_0402_1005Metric
- removed C30: 1.2pF, Capacitor_SMD:C_0402_1005Metric
- removed the D23 at (122.3, 121.5)
- removed the D24 at (104.2, 115.9)
- removed the D25 at (86.2, 110.2)
- removed the D26 at (68.2, 115.9)
- removed the D27 at (50.2, 121.5)
- removed the D28 at (122.3, 104.5)
- removed the D29 at (104.3, 98.8)
- removed the D30 at (86.2, 93.2)
- removed the D31 at (68.2, 98.8)
- removed the D32 at (50.2, 104.5)
- removed the D33 at (122.2, 87.5)
- removed the D34 at (104.3, 81.8)
- removed the D35 at (86.3, 76.2)
- removed the D36 at (68.3, 81.8)
- removed the D37 at (50.2, 87.5)
- removed the D38 at (122.2, 70.5)
- removed the D39 at (104.2, 64.8)
- removed the D40 at (86.2, 59.2)
- removed the D41 at (68.2, 64.8)
- removed the D42 at (50.3, 70.5)
- removed D43, D44, D45, D46, D47, D48, D49, D50, D51, D52, D53, D54, D55, D56, D57, D58, D59, D60, D61, D62, D63, D64: 1N5819, Diode_SMD:D_SOD-123
- removed D65, D66, D67, D68, D69, D70, D71, D72, D73, D74, D75, D76, D77, D78, D79, D80, D81, D82, D83, D84: SK6812MINI, Keebio_Parts:SK6812-MINI-E
- removed F2: 500mA, Fuse:Fuse_0603_1608Metric
- removed H10, H6, H7, H8, H9: MountingHole, MountingHole:MountingHole_2mm
- removed J4: Conn_01x02, Connector_PinHeader_1.00mm:PinHeader_1x02_P1.00mm_Vertical
- removed J5: SWD_Connector, Connector_PinHeader_1.00mm:PinHeader_1x04_P1.00mm_Vertical
- removed J6: USB_C_Receptacle_USB2.0_14P, USB_Type_C:HRO-TYPE-C-31-M-12
- removed L10: 2.2nH, Inductor_SMD:L_0201_0603Metric
- removed L6, L8: 10uH, Inductor_SMD:L_1008_2520Metric
- removed L7: 15nH, Inductor_SMD:L_0201_0603Metric
- removed L9: 4.7nH, Inductor_SMD:L_0201_0603Metric
- removed Q2: BSS138, Package_TO_SOT_SMD:SOT-23
- removed R10, R13, R14, R9: 10K, Resistor_SMD:R_0201_0603Metric
- removed R11, R12: 5.1k, Resistor_SMD:R_0201_0603Metric
- removed R8: 100K, Resistor_SMD:R_0201_0603Metric
- removed SW24: SW_On_Off, Button_Switch_THT:SW_CK_JS202011AQN_DPDT_Angled
- removed SW25, SW26, SW27, SW28, SW29, SW31, SW32, SW33, SW34, SW35, SW36, SW37, SW38, SW39, SW40, SW41, SW42, SW43, SW44, SW45: SW_Push, PCM_Switch_Keyboard_Hotswap_Kailh:SW_Hotswap_Kailh_Choc_V1V2_1.00u
- removed SW30: Reset Button, Button_Switch_SMD:SW_SPST_TL3342
- removed SW46: SW_Push, PCM_Switch_Keyboard_Hotswap_Kailh:SW_Hotswap_Kailh_Choc_V1V2_1.75u_90deg
- removed U4: nRF52840, Package_DFN_QFN:Nordic_AQFN-73-1EP_7x7mm_P0.5mm
- removed U5: USBLC6-2SC6, Package_TO_SOT_SMD:SOT-23-6
- removed U6: AMS1117-5.0, Package_TO_SOT_SMD:SOT-223-3_TabPin2
- removed Y2: JYJE 2TJ432000NYFBC, Crystal:Crystal_SMD_2520-4Pin_2.5x2.0mm
- D24, D25, D26, D28, D29, D30, D31, D32, D33, D34, D35, D36, D37, D38, D39, D40, D41, D42: moved to B.Cu
- moved D42 336.4 mm to (47.6, 70.8), turned to 180 degrees
- moved D37 324.7 mm to (47.7, 87.9)
- moved D41 319.3 mm to (65.6, 65.1), turned to 180 degrees
- moved D32 313.9 mm to (47.6, 104.8), turned to 180 degrees
- moved D36 307.3 mm to (65.7, 82.2)
- moved D27 304.2 mm to (47.6, 121.8), turned to 0 degrees
- moved D40 302.3 mm to (83.6, 59.4), turned to 180 degrees
- moved D31 296.3 mm to (65.6, 99.1), turned to 180 degrees
- moved D35 290.2 mm to (83.6, 76.4)
- moved D26 286.0 mm to (65.6, 116.1)
- moved D39 282.2 mm to (101.6, 65.1), turned to 180 degrees
- moved D30 275.8 mm to (86.7, 93.5), turned to 180 degrees
- moved D34 270.2 mm to (101.7, 82.2)
- moved D25 268.3 mm to (83.6, 110.4)
- moved D38 261.9 mm to (119.7, 70.9), turned to 180 degrees
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- renumbered D2 to D1, SW1 to SW2
Connections:
- net /ANT renamed /left/ANT
- net /BT_PIN renamed /left/BT_PIN
- net /CC1 renamed /left/CC1
- net /CC2 renamed /left/CC2
- net /COL0 renamed /left/COL0
- net /COL1 renamed /left/COL1
- net /COL2 renamed /left/COL2
- net /COL3 renamed /left/COL3
- net /COL4 renamed /left/COL4
- net /D+ renamed /left/D+
- net /D- renamed /left/D-
- net /DCC renamed /left/DCC
- net /DCCH renamed /left/DCCH
- net /DEC1 renamed /left/DEC1
- net /DEC3 renamed /left/DEC3
- net /DEC4 renamed /left/DEC4
- net /DEC5 renamed /left/DEC5
- net /DECUSB renamed /left/DECUSB
- net /RESET renamed /left/RESET
- net /ROW0 renamed /left/ROW0
- net /ROW1 renamed /left/ROW1
- net /ROW2 renamed /left/ROW2
- net /ROW3 renamed /left/ROW3
- net /ROW4 renamed /left/ROW4
- net /SWDCLK renamed /left/SWDCLK
- net /SWDIO renamed /left/SWDIO
- net /XC1 renamed /left/XC1
- net /XC2 renamed /left/XC2
- Q1 pad 2: LED_PIN -> /left/leds/LED_PIN
- Q1 pad 3: /leds/DATA -> /left/leds/DATA
- R6 pad 2: LED_PIN -> /left/leds/LED_PIN
- R7 pad 2: /leds/DATA -> /left/leds/DATA
- U1 pad A12: LED_PIN -> /left/LED_PIN
Routing:
- net LED_5V: track 433.9 -> 29.8 mm, vias 6 -> 4
- net GND: track 654.0 -> 311.5 mm, vias 22 -> 13
- net V_SYS: track 142.3 -> 5.65 mm, vias 12 -> 0
- net /left/COL3: track 124.1 -> 41.7 mm, vias 4 -> 3
- net /left/COL1: track 162.2 -> 102.8 mm, vias 8 -> 5
- net LED_PIN: track 35.3 -> 0.00 mm, vias 2 -> 0
- net /left/leds/LED_PIN: track 0.00 -> 35.3 mm, vias 0 -> 2
- net /left/SWDIO: track 84.7 -> 49.9 mm, vias 6 -> 4
- net /leds/DATA: track 34.3 -> 0.00 mm, vias 2 -> 0
- net Net-(D28-DOUT): track 24.3 -> 0.00 mm
- net Net-(D33-DOUT): track 23.6 -> 0.00 mm, vias 2 -> 0
- net VBAT: track 88.5 -> 66.7 mm, vias 6 -> 5
- net Net-(D39-DIN): track 20.8 -> 0.00 mm
- net Net-(D28-DIN): track 20.6 -> 0.00 mm
- net VBUS: track 93.6 -> 73.0 mm, vias 6 -> 4
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